File: Washingboard.kicad_sch (KiCad schematic)
At the start: 21 parts, among them CN1 JST S2B-PH-SM4-TB(LF)(SN), J2 USB_C_Receptacle_USB2.0_14P, Q1 DMP2045UQ-7, SW1 SW_Push, SW2 SW_Push, U1 RT9080-33GJ5, U2 ESP32-S3-MINI-1

Commit message: PCB Layout
Parts:
- removed SW1, SW2: SW_Push, symbol Switch:SW_Push
- added C6: 10uF, Capacitor_SMD:C_0805_2012Metric, symbol Device:C
- added LED1: FC-2012HRK-620D, easyeda2kicad:LED0805-R-RD, symbol easyeda2kicad:FC-2012HRK-620D
- added R10, R8, R9: 5.1K, Resistor_SMD:R_0805_2012Metric, symbol Device:R
- added R11: 160, Resistor_SMD:R_0805_2012Metric, symbol Device:R
- added R12: 2k, Resistor_SMD:R_0805_2012Metric, symbol Device:R
- added SW1, SW2: TS-1088-AR02016, easyeda2kicad:SW-SMD_L3.9-W3.0-P4.45, symbol easyeda2kicad:TS-1088-AR02016
- added U3: LIS3DHTR_C15134, easyeda2kicad:LGA-16_L3.0-W3.0-P0.50-TL, symbol easyeda2kicad:LIS3DHTR_C15134
- added U4: MCP73831T-2ACI/OT, easyeda2kicad:SOT-23-5_L3.0-W1.7-P0.95-LS2.8-BL, symbol easyeda2kicad:MCP73831T-2ACI_OT
- C4: value 10uF -> 0.1uF; LCSC Part C1713 -> C1711
- J2: value USB_C_Receptacle_USB2.0_14P -> HCTL HC-TYPE-C-16P-01A
- R5: value 100K -> 470K; LCSC Part C25611 -> C17709
- R6: value 348K -> 470K; LCSC Part C17638 -> C17709
Connections:
- net 3.3V: now also R10.2, R8.2, R9.2, U3.1 (VDD_IO), U3.14 (VDD)
- net BOOT: now also SW2.2
- net GND: now also J2.A1 (GND), J2.A12 (GND), J2.B1 (GND), J2.B12 (GND), J2.S1 (SHIELD), C6.2, R12.2, SW1.1, SW2.1, U3.10 (RES), U3.12 (GND), U3.5 (GND), U4.2 (VSS)
- net GPIO1: now also U2.15 (IO11); no longer U2.5 (IO1)
- net RESET: now also SW1.2
- net VBAT: now also C6.1, U4.3 (VBAT)
- net VBUS: now also Q1.1 (G), R11.1, U4.4 (VDD); no longer C1.1, D1.1 (K), Q1.2 (S), R2.1, U1.1 (VIN)
- net INT1: now reaches U2.31 (IO35)
- net INT1: now also U3.11 (INT1)
- net SCL: now reaches U2.32 (IO36)
- net SCL: now also R10.1, U3.4 (SCL/SPC)
- net SDA: now reaches U2.33 (IO37)
- net SDA: now also R9.1, U3.6 (SDA/SDI/SDO)
- new net: C1.1, D1.1 (K), Q1.2 (S), R2.1, U1.1 (VIN)
- new net: R8.1, U3.8 (CS)
- new net: LED1.2 (-), U4.1 (STAT)
- new net: R12.1, U4.5 (PROG)
- new net: LED1.1 (+), R11.2
- no-connect marks 0 -> 42
Other:
- note added: "1.0"
- note added: "11/02/2024"
- note added: "Wakeboard"
- moved on the sheet: C2, C3, C4, U2
